Commit message: 4.0.0: Versio final de codi validada en simulació

File: src/car_simulator/urdf/car.urdf (robot description, URDF)
Before this commit: robot car, 2 links, 1 joints
Links:
- added link front_left_wheel; visual cylinder length=0.026 radius=0.0325; visual cylinder length=0.027 radius=0.020
- added link front_right_wheel; visual cylinder length=0.026 radius=0.0325; visual cylinder length=0.027 radius=0.020
- added link rear_left_wheel; visual cylinder length=0.026 radius=0.0325; visual cylinder length=0.027 radius=0.020
- added link rear_right_wheel; visual cylinder length=0.026 radius=0.0325; visual cylinder length=0.027 radius=0.020
- link base_link: geometry collision box size=0.33 0.13 0.06; visual box size=0.004 0.110 0.005
- link ldlidar_base: geometry visual cylinder length=0.035 radius=0.019
Joints:
- added joint front_left_steer_joint: type revolute, parent base_link, child front_left_wheel, origin xyz=0 0.065 0.0325 rpy=0 0 0, axis 0 0 1, limit lower=-0.8 upper=0.8 effort=1.0 velocity=10.0
- added joint front_right_steer_joint: type revolute, parent base_link, child front_right_wheel, origin xyz=0 -0.065 0.0325 rpy=0 0 0, axis 0 0 1, limit lower=-0.8 upper=0.8 effort=1.0 velocity=10.0
- added joint rear_left_wheel_joint: type fixed, parent base_link, child rear_left_wheel, origin xyz=-0.18 0.065 0.0325 rpy=0 0 0
- added joint rear_right_wheel_joint: type fixed, parent base_link, child rear_right_wheel, origin xyz=-0.18 -0.065 0.0325 rpy=0 0 0
- joint lidar_mount_joint: origin xyz=0 0 0.12 rpy=0 0 0 -> xyz=0 0 0.085 rpy=0 0 0

Commit message: Solucio error primeres proves

File: src/car_simulator/urdf/car.urdf (robot description, URDF)
Before this commit: robot car, 6 links, 5 joints
Joints:
- joint front_left_steer_joint: limit lower=-0.8 upper=0.8 effort=1.0 velocity=10.0 -> lower=-0.4062 upper=0.4062 effort=1.0 velocity=10.0
- joint front_right_steer_joint: limit lower=-0.8 upper=0.8 effort=1.0 velocity=10.0 -> lower=-0.4062 upper=0.4062 effort=1.0 velocity=10.0
